Commit message: add the URDF of a robot

File: ouster_ros/urdf/my_robot_2d.urdf (robot description, URDF)
Before this commit: robot anyName_2D, 5 links, 4 joints
Joints:
- joint base_link_imu_joint: origin xyz=0.60 0 0.88 rpy=0 0 0 -> xyz=0.0 0 0.88 rpy=0 0 0
- joint base_link_laser_joint: origin xyz=0.60 0 0.88 rpy=0 0 0 -> xyz=0.0 0 0.88 rpy=0 0 0
